Commit message: Import all sensor tools CAD and rename STL files for readability. Added lookup documentation

File: src/meca500_scene_description/urdf/scene.urdf.xacro (robot description, xacro)
@@ -3,5 +3,5 @@
   <!-- Trusted Meca500 robot model -->
   <xacro:include filename="$(find meca500_description)/urdf/meca500_macro.xacro"/>
-  <!-- Global reference frame for Dio's bench CAD -->
+  <!-- Global reference frame for the Helico bench CAD -->
   <link name="world"/>
   <link name="bench_frame"/>
@@ -12,10 +12,10 @@
   </joint>
   <!--
-    Dio bench breadboard.
+    Helico bench breadboard.
     This mesh comes from the original Onshape URDF export and is the
     authoritative geometric reference for positioning the physical bench.
     No manually tuned RViz offset is applied here.
   -->
-  <link name="dio_breadboard">
+  <link name="bench_breadboard">
     <visual>
       <origin xyz="0 -0.0127 0" rpy="0 0 0"/>
@@ -29,12 +29,76 @@
   </link>
   <!-- ========================================================= -->
-  <!-- Helico fixture bases                                      -->
-  <!--                                                          -->
-  <!-- Derived directly from Dio's Onshape URDF.                -->
-  <!-- Original Onshape names: base, base_1, base_2.            -->
-  <!-- Renamed here to avoid ambiguous CAD-generated names.     -->
-  <!-- ========================================================= -->
-  <!-- Fixture 1 -->
-  <link name="fixture_1_base">
+  <!-- Helico balloon tip stations                              -->
+  <!--                                                          -->
+  <!-- Ordered physically from robot-right to robot-left:        -->
+  <!--   3.5 mm -> 4 mm -> 5 mm                                 -->
+  <!--                                                          -->
+  <!-- Helico CAD mapping:                                         -->
+  <!--   base_1 -> 3.5 mm station                               -->
+  <!--   base   -> 4 mm station                                 -->
+  <!--   base_2 -> 5 mm station                                 -->
+  <!-- ========================================================= -->
+  <!-- ========================================================= -->
+  <!-- 3.5 mm tip station                                       -->
+  <!-- Robot-right station                                      -->
+  <!-- Helico CAD source: base_1                                   -->
+  <!-- ========================================================= -->
+  <link name="tip_station_3p5mm_base">
+    <visual>
+      <origin xyz="-0.0125 0.0125 0.025" rpy="0 0 0"/>
+      <geometry>
+        <mesh filename="package://meca500_scene_description/meshes/onshape/Base.stl"/>
+      </geometry>
+    <material name="base_colour">
+      <color rgba="0.4 0.7 0.9 1.0"/>
+    </material>
+    </visual>
+  </link>
+  <joint name="breadboard_to_tip_station_3p5mm_base" type="fixed">
+    <parent link="bench_breadboard"/>
+    <child link="tip_station_3p5mm_base"/>
+    <origin xyz="-0.0125 -0.0127 -0.0875"
+            rpy="1.5708 0 0"/>
+  </joint>
+  <link name="tip_station_3p5mm_coupling_base">
+    <visual>
+      <origin xyz="-0.006 0 0" rpy="0 0 0"/>
+      <geometry>
+        <mesh filename="package://meca500_scene_description/meshes/onshape/Coupling_base.stl"/>
+      </geometry>
+    <material name="coupling_colour">
+      <color rgba="0.1 0.3 0.8 1.0"/>
+    </material>
+    </visual>
+  </link>
+  <joint name="tip_station_3p5mm_base_to_coupling_base" type="fixed">
+    <parent link="tip_station_3p5mm_base"/>
+    <child link="tip_station_3p5mm_coupling_base"/>
+    <origin xyz="-0.0065 0.0125 0.025"
+            rpy="0 0 0"/>
+  </joint>
+  <link name="tip_station_3p5mm_holder">
+    <visual>
+      <origin xyz="0 0 0" rpy="0 0 0"/>
+      <geometry>
+        <mesh filename="package://meca500_scene_description/meshes/onshape/_3D_printed.stl"/>
+      </geometry>
+    <material name="holder_colour">
+      <color rgba="0.9 0.1 0.1 1.0"/>
+    </material>
+    </visual>
+  </link>
+  <joint name="tip_station_3p5mm_coupling_base_to_holder" type="fixed">
+    <parent link="tip_station_3p5mm_coupling_base"/>
+    <child link="tip_station_3p5mm_holder"/>
+    <origin xyz="-0.006 0 0.005"
+            rpy="-1.5708 0 1.5708"/>
+  </joint>
+  <!-- ========================================================= -->
+  <!-- 4 mm tip station                                         -->
+  <!-- Middle station                                           -->
+  <!-- Helico CAD source: base -> coupling_base_1 -> 3d_printed_1  -->
+  <!-- ========================================================= -->
+  <link name="tip_station_4mm_base">
     <visual>
       <origin xyz="0.0125 0.0125 0.025" rpy="0 0 0"/>
@@ -42,14 +106,55 @@
         <mesh filename="package://meca500_scene_description/meshes/onshape/Base.stl"/>
       </geometry>
-    </visual>
-  </link>
-  <joint name="breadboard_to_fixture_1_base" type="fixed">
-    <parent link="dio_breadboard"/>
-    <child link="fixture_1_base"/>
+    <material name="base_colour">
+      <color rgba="0.4 0.7 0.9 1.0"/>
+    </material>
+    </visual>
+  </link>
+  <joint name="breadboard_to_tip_station_4mm_base" type="fixed">
+    <parent link="bench_breadboard"/>
+    <child link="tip_station_4mm_base"/>
     <origin xyz="-0.0375 -0.0127 -0.0125"
             rpy="1.5708 0 0"/>
   </joint>
-  <!-- Fixture 2 -->
-  <link name="fixture_2_base">
+  <link name="tip_station_4mm_coupling_base">
+    <visual>
+      <origin xyz="-0.006 0 0" rpy="0 0 0"/>
+      <geometry>
+        <mesh filename="package://meca500_scene_description/meshes/onshape/Coupling_base.stl"/>
+      </geometry>
+    <material name="coupling_colour">
+      <color rgba="0.1 0.3 0.8 1.0"/>
+    </material>
+    </visual>
+  </link>
+  <joint name="tip_station_4mm_base_to_coupling_base" type="fixed">
+    <parent link="tip_station_4mm_base"/>
+    <child link="tip_station_4mm_coupling_base"/>
+    <origin xyz="0.0185 0.0125 0.025"
+            rpy="0 0 0"/>
+  </joint>
+  <link name="tip_station_4mm_holder">
+    <visual>
+      <origin xyz="0 -0.0123 0" rpy="0 0 0"/>
+      <geometry>
+        <mesh filename="package://meca500_scene_description/meshes/onshape/_3D_printed.stl"/>
+      </geometry>
+    <material name="holder_colour">
+      <color rgba="0.9 0.1 0.1 1.0"/>
+    </material>
+    </visual>
+  </link>
+  <joint name="tip_station_4mm_coupling_base_to_holder" type="fixed">
+    <parent link="tip_station_4mm_coupling_base"/>
+    <child link="tip_station_4mm_holder"/>
+    <origin xyz="-0.006 0 0.005"
+            rpy="-1.5708 0 1.5708"/>
+  </joint>
+  <!-- ========================================================= -->
+  <!-- 5 mm tip station                                         -->
+  <!-- Robot-left station                                       -->
+  <!-- Helico CAD source: base_2                                   -->
+  <!-- ========================================================= -->
+  <link name="tip_station_5mm_base">
     <visual>
       <origin xyz="-0.0125 0.0125 0.025" rpy="0 0 0"/>
@@ -57,24 +162,12 @@
         <mesh filename="package://meca500_scene_description/meshes/onshape/Base.stl"/>
       </geometry>
-    </visual>
-  </link>
-  <joint name="breadboard_to_fixture_2_base" type="fixed">
-    <parent link="dio_breadboard"/>
-    <child link="fixture_2_base"/>
-    <origin xyz="-0.0125 -0.0127 -0.0875"
-            rpy="1.5708 0 0"/>
-  </joint>
-  <!-- Fixture 3 -->
-  <link name="fixture_3_base">
-    <visual>
-      <origin xyz="-0.0125 0.0125 0.025" rpy="0 0 0"/>
-      <geometry>
-        <mesh filename="package://meca500_scene_description/meshes/onshape/Base.stl"/>
-      </geometry>
-    </visual>
-  </link>
-  <joint name="breadboard_to_fixture_3_base" type="fixed">
-    <parent link="dio_breadboard"/>
-    <child link="fixture_3_base"/>
+    <material name="base_colour">
+      <color rgba="0.4 0.7 0.9 1.0"/>
+    </material>
+    </visual>
+  </link>
+  <joint name="breadboard_to_tip_station_5mm_base" type="fixed">
+    <parent link="bench_breadboard"/>
+    <child link="tip_station_5mm_base"/>
     <origin xyz="-0.0125 -0.0127 0.0625"
             rpy="1.5708 0 0"/>
@@ -82,11 +175,11 @@
 <joint name="bench_to_breadboard" type="fixed">
   <parent link="bench_frame"/>
-  <child link="dio_breadboard"/>
+  <child link="bench_breadboard"/>
   <origin xyz="0 0 0" rpy="-1.5708 0 0"/>
 </joint>
-<xacro:meca500 parent="dio_breadboard">
+<xacro:meca500 parent="bench_breadboard">
   <!--
-    Trusted ROS Meca500 kinematic model positioned using Dio's CAD.
-    Placement derived from rigid registration of Dio's Base_1.stl
+    Trusted ROS Meca500 kinematic model positioned using Helico's CAD.
+    Placement derived from rigid registration of Helico's Base_1.stl
     against the trusted ROS Meca500 base mesh.
     Do not tune this transform manually in RViz.
@@ -95,4 +188,136 @@
           rpy="1.5708 0 0"/>
 </xacro:meca500>
+  <!-- ========================================================= -->
+  <!-- Link 6 measurement tool                                  -->
+  <!--                                                          -->
+  <!-- Physical instrument geometry derived from the Onshape    -->
+  <!-- assembly. Only real fixed CAD components are represented. -->
+  <!--                                                          -->
+  <!-- CAD mapping:                                             -->
+  <!--   l6         -> link_6                                   -->
+  <!--   part_1_2   -> tools_mount                              -->
+  <!--   part_1   -> laser_sensor_mount                         -->
+  <!--   8777405    -> laser_sensor                             -->
+  <!--   Force_sensor -> force_sensor                           -->
+  <!--   part_1_3   -> april_tag_mount                          -->
+  <!--   part_1_10   -> force_poker                             -->
+  <!--                                                          -->
+  <!-- NOTE: link_6 <-> CAD l6 frame equivalence must be        -->
+  <!-- physically verified before real robot operation.         -->
+  <!-- ========================================================= -->
+  <!-- Main tool mounting body -->
+  <link name="tools_mount">
+    <visual>
+      <origin xyz="-0.00548008 0 -0.00548008"
+              rpy="0 0 0"/>
+      <geometry>
+        <mesh filename="package://meca500_scene_description/meshes/onshape/tools_mount.stl"/>
+      </geometry>
+      <material name="tools_mount_colour">
+        <color rgba="0.682353 0.333333 0.737255 1"/>
+      </material>
+    </visual>
+  </link>
+  <joint name="link_6_to_tools_mount" type="fixed">
+    <parent link="link_6"/>
+    <child link="tools_mount"/>
+    <origin xyz="-0.00548008 0.00548008 0"
+            rpy="-1.5708 0 1.5708"/>
+  </joint>
+  <!-- Laser mounting/support component -->
+  <link name="laser_sensor_mount">
+    <visual>
+      <origin xyz="-0.00273616 -0.00751754 -0.0575"
+              rpy="0 0 0"/>
+      <geometry>
+        <mesh filename="package://meca500_scene_description/meshes/onshape/laser_sensor_mount.stl"/>
+      </geometry>
+      <material name="laser_sensor_mount_colour">
+        <color rgba="0.729412 0.25098 0.105882 1"/>
+      </material>
+    </visual>
+  </link>
+  <joint name="tools_mount_to_laser_sensor_mount" type="fixed">
+    <parent link="tools_mount"/>
+    <child link="laser_sensor_mount"/>
+    <origin xyz="0.00203746 -0.005 0.0247125"
+            rpy="0 -1.5708 -1.5708"/>
+  </joint>
+  <!-- Laser displacement sensor -->
+  <link name="laser_sensor">
+    <visual>
+      <origin xyz="-0.01 -0.0028 0.0215"
+              rpy="0 0 0"/>
+      <geometry>
+        <mesh filename="package://meca500_scene_description/meshes/onshape/laser_sensor.stl"/>
+      </geometry>
+      <material name="laser_sensor_colour">
+        <color rgba="0.615686 0.811765 0.929412 1"/>
+      </material>
+    </visual>
+  </link>
+  <joint name="laser_sensor_mount_to_laser_sensor" type="fixed">
+    <parent link="laser_sensor_mount"/>
+    <child link="laser_sensor"/>
+    <origin xyz="0.0320138 -0.0100175 -0.0828716"
+            rpy="-1.5708 0 1.5708"/>
+  </joint>
+  <!-- Force sensor body -->
+  <link name="force_sensor">
+    <visual>
+      <origin xyz="0.0277 0 0"
+              rpy="0 0 0"/>
+      <geometry>
+        <mesh filename="package://meca500_scene_description/meshes/onshape/force_sensor.stl"/>
+      </geometry>
+      <material name="force_sensor_colour">
+        <color rgba="0.901961 0.901961 0.901961 1"/>
+      </material>
+    </visual>
+  </link>
+  <joint name="tools_mount_to_force_sensor" type="fixed">
+    <parent link="tools_mount"/>
+    <child link="force_sensor"/>
+    <origin xyz="-0.00548008 -0.019 -0.0424801"
+            rpy="0 -1.5708 3.14159"/>
+  </joint>
+  <!-- Force poker -->
+  <link name="force_poker">
+    <visual>
+      <origin xyz="-0.004 0 -0.03375"
+              rpy="0 0 0"/>
+      <geometry>
+        <mesh filename="package://meca500_scene_description/meshes/onshape/force_poker.stl"/>
+      </geometry>
+      <material name="force_poker_colour">
+        <color rgba="0.282353 0.54902 0.160784 1"/>
+      </material>
+    </visual>
+  </link>
+  <joint name="force_sensor_to_force_poker" type="fixed">
+    <parent link="force_sensor"/>
+    <child link="force_poker"/>
+    <origin xyz="0.0168 0 0"
+            rpy="-1.5708 0 -3.14159"/>
+  </joint>
+  <!-- April Tag mount -->
+  <link name="april_tag_mount">
+    <visual>
+      <origin xyz="0 0.01 0"
+              rpy="0 0 0"/>
+      <geometry>
+        <mesh filename="package://meca500_scene_description/meshes/onshape/april_tag_mount.stl"/>
+      </geometry>
+      <material name="april_tag_mount_colour">
+        <color rgba="0.980392 0.713726 0.00392157 1"/>
+      </material>
+    </visual>
+  </link>
+  <joint name="tools_mount_to_april_tag_mount" type="fixed">
+    <parent link="tools_mount"/>
+    <child link="april_tag_mount"/>
+    <origin xyz="-0.0419365 -0.0025 -0.0154801"
+            rpy="1.5708 0 -1.5708"/>
+  </joint>
   <!-- ========================================================= -->
   <!-- Mock ros2_control                                         -->
