Commit message: Add bench and tool collision geometry with SRDF collision exclusions

File: src/meca500_scene_description/urdf/scene.urdf.xacro (robot description, xacro)
@@ -27,4 +27,10 @@
       </material>
     </visual>
+    <collision>
+      <origin xyz="0 -0.0127 0" rpy="0 0 0"/>
+      <geometry>
+        <mesh filename="package://meca500_scene_description/meshes/onshape/MB3060_M___Aluminium_Breadboard_300_x_600_x_12_7mm_MB3030_M_1.stl"/>
+      </geometry>
+    </collision>
   </link>
   <!-- ========================================================= -->
@@ -34,13 +40,19 @@
   <!--   3.5 mm -> 4 mm -> 5 mm                                 -->
   <!--                                                          -->
-  <!-- Helico CAD mapping:                                         -->
-  <!--   base_1 -> 3.5 mm station                               -->
-  <!--   base   -> 4 mm station                                 -->
-  <!--   base_2 -> 5 mm station                                 -->
-  <!-- ========================================================= -->
-  <!-- ========================================================= -->
-  <!-- 3.5 mm tip station                                       -->
-  <!-- Robot-right station                                      -->
-  <!-- Helico CAD source: base_1                                   -->
+  <!-- Current station geometry is a PLACEHOLDER representation. -->
+  <!-- Repeated CAD meshes are used where the final Onshape CAD  -->
+  <!-- has not yet been completed.                               -->
+  <!--                                                          -->
+  <!-- Final station geometry should be updated from the latest  -->
+  <!-- Onshape assembly when available.                          -->
+  <!--                                                          -->
+  <!-- Helico CAD mapping:                                       -->
+  <!--   base_1 -> 3.5 mm station                                -->
+  <!--   base   -> 4 mm station                                  -->
+  <!--   base_2 -> 5 mm station                                  -->
+  <!-- ========================================================= -->
+  <!-- ========================================================= -->
+  <!-- 3.5 mm tip station                                        -->
+  <!-- Robot-right station                                       -->
   <!-- ========================================================= -->
   <link name="tip_station_3p5mm_base">
@@ -50,8 +62,14 @@
         <mesh filename="package://meca500_scene_description/meshes/onshape/Base.stl"/>
       </geometry>
-    <material name="base_colour">
-      <color rgba="0.4 0.7 0.9 1.0"/>
-    </material>
-    </visual>
+      <material name="base_colour">
+        <color rgba="0.4 0.7 0.9 1.0"/>
+      </material>
+    </visual>
+    <collision>
+      <origin xyz="-0.0125 0.0125 0.025" rpy="0 0 0"/>
+      <geometry>
+        <mesh filename="package://meca500_scene_description/meshes/onshape/Base.stl"/>
+      </geometry>
+    </collision>
   </link>
   <joint name="breadboard_to_tip_station_3p5mm_base" type="fixed">
@@ -67,8 +85,14 @@
         <mesh filename="package://meca500_scene_description/meshes/onshape/Coupling_base.stl"/>
       </geometry>
-    <material name="coupling_colour">
-      <color rgba="0.1 0.3 0.8 1.0"/>
-    </material>
-    </visual>
+      <material name="coupling_colour">
+        <color rgba="0.1 0.3 0.8 1.0"/>
+      </material>
+    </visual>
+    <collision>
+      <origin xyz="-0.006 0 0" rpy="0 0 0"/>
+      <geometry>
+        <mesh filename="package://meca500_scene_description/meshes/onshape/Coupling_base.stl"/>
+      </geometry>
+    </collision>
   </link>
   <joint name="tip_station_3p5mm_base_to_coupling_base" type="fixed">
@@ -80,12 +104,18 @@
   <link name="tip_station_3p5mm_holder">
     <visual>
-      <origin xyz="0 0 0" rpy="0 0 0"/>
-      <geometry>
-        <mesh filename="package://meca500_scene_description/meshes/onshape/_3D_printed.stl"/>
-      </geometry>
-    <material name="holder_colour">
-      <color rgba="0.9 0.1 0.1 1.0"/>
-    </material>
-    </visual>
+      <origin xyz="0 -0.0123 0" rpy="0 0 0"/>
+      <geometry>
+        <mesh filename="package://meca500_scene_description/meshes/onshape/_3D_printed.stl"/>
+      </geometry>
+      <material name="holder_colour">
+        <color rgba="0.95 0.75 0.20 1.0"/>
+      </material>
+    </visual>
+    <collision>
+      <origin xyz="0 -0.0123 0" rpy="0 0 0"/>
+      <geometry>
+        <mesh filename="package://meca500_scene_description/meshes/onshape/_3D_printed.stl"/>
+      </geometry>
+    </collision>
   </link>
   <joint name="tip_station_3p5mm_coupling_base_to_holder" type="fixed">
@@ -96,7 +126,6 @@
   </joint>
   <!-- ========================================================= -->
-  <!-- 4 mm tip station                                         -->
-  <!-- Middle station                                           -->
-  <!-- Helico CAD source: base -> coupling_base_1 -> 3d_printed_1  -->
+  <!-- 4 mm tip station                                          -->
+  <!-- Middle station                                            -->
   <!-- ========================================================= -->
   <link name="tip_station_4mm_base">
@@ -106,8 +135,14 @@
         <mesh filename="package://meca500_scene_description/meshes/onshape/Base.stl"/>
       </geometry>
-    <material name="base_colour">
-      <color rgba="0.4 0.7 0.9 1.0"/>
-    </material>
-    </visual>
+      <material name="base_colour">
+        <color rgba="0.4 0.7 0.9 1.0"/>
+      </material>
+    </visual>
+    <collision>
+      <origin xyz="0.0125 0.0125 0.025" rpy="0 0 0"/>
+      <geometry>
+        <mesh filename="package://meca500_scene_description/meshes/onshape/Base.stl"/>
+      </geometry>
+    </collision>
   </link>
   <joint name="breadboard_to_tip_station_4mm_base" type="fixed">
@@ -123,8 +158,14 @@
         <mesh filename="package://meca500_scene_description/meshes/onshape/Coupling_base.stl"/>
       </geometry>
-    <material name="coupling_colour">
-      <color rgba="0.1 0.3 0.8 1.0"/>
-    </material>
-    </visual>
+      <material name="coupling_colour">
+        <color rgba="0.1 0.3 0.8 1.0"/>
+      </material>
+    </visual>
+    <collision>
+      <origin xyz="-0.006 0 0" rpy="0 0 0"/>
+      <geometry>
+        <mesh filename="package://meca500_scene_description/meshes/onshape/Coupling_base.stl"/>
+      </geometry>
+    </collision>
   </link>
   <joint name="tip_station_4mm_base_to_coupling_base" type="fixed">
@@ -140,8 +181,14 @@
         <mesh filename="package://meca500_scene_description/meshes/onshape/_3D_printed.stl"/>
       </geometry>
-    <material name="holder_colour">
-      <color rgba="0.9 0.1 0.1 1.0"/>
-    </material>
-    </visual>
+      <material name="holder_colour">
+        <color rgba="0.95 0.75 0.20 1.0"/>
+      </material>
+    </visual>
+    <collision>
+      <origin xyz="0 -0.0123 0" rpy="0 0 0"/>
+      <geometry>
+        <mesh filename="package://meca500_scene_description/meshes/onshape/_3D_printed.stl"/>
+      </geometry>
+    </collision>
   </link>
   <joint name="tip_station_4mm_coupling_base_to_holder" type="fixed">
@@ -152,7 +199,9 @@
   </joint>
   <!-- ========================================================= -->
-  <!-- 5 mm tip station                                         -->
-  <!-- Robot-left station                                       -->
-  <!-- Helico CAD source: base_2                                   -->
+  <!-- 5 mm tip station                                          -->
+  <!-- Robot-left station                                        -->
+  <!--                                                          -->
+  <!-- PLACEHOLDER: coupling and holder reuse the existing        -->
+  <!-- station meshes until final Onshape CAD is available.       -->
   <!-- ========================================================= -->
   <link name="tip_station_5mm_base">
@@ -162,8 +211,14 @@
         <mesh filename="package://meca500_scene_description/meshes/onshape/Base.stl"/>
       </geometry>
-    <material name="base_colour">
-      <color rgba="0.4 0.7 0.9 1.0"/>
-    </material>
-    </visual>
+      <material name="base_colour">
+        <color rgba="0.4 0.7 0.9 1.0"/>
+      </material>
+    </visual>
+    <collision>
+      <origin xyz="-0.0125 0.0125 0.025" rpy="0 0 0"/>
+      <geometry>
+        <mesh filename="package://meca500_scene_description/meshes/onshape/Base.stl"/>
+      </geometry>
+    </collision>
   </link>
   <joint name="breadboard_to_tip_station_5mm_base" type="fixed">
@@ -173,9 +228,59 @@
             rpy="1.5708 0 0"/>
   </joint>
-<joint name="bench_to_breadboard" type="fixed">
-  <parent link="bench_frame"/>
-  <child link="bench_breadboard"/>
-  <origin xyz="0 0 0" rpy="-1.5708 0 0"/>
-</joint>
+  <link name="tip_station_5mm_coupling_base">
+    <visual>
+      <origin xyz="-0.006 0 0" rpy="0 0 0"/>
+      <geometry>
+        <mesh filename="package://meca500_scene_description/meshes/onshape/Coupling_base.stl"/>
+      </geometry>
+      <material name="coupling_colour">
+        <color rgba="0.1 0.3 0.8 1.0"/>
+      </material>
+    </visual>
+    <collision>
+      <origin xyz="-0.006 0 0" rpy="0 0 0"/>
+      <geometry>
+        <mesh filename="package://meca500_scene_description/meshes/onshape/Coupling_base.stl"/>
+      </geometry>
+    </collision>
+  </link>
+  <joint name="tip_station_5mm_base_to_coupling_base" type="fixed">
+    <parent link="tip_station_5mm_base"/>
+    <child link="tip_station_5mm_coupling_base"/>
+    <origin xyz="-0.0065 0.0125 0.025"
+            rpy="0 0 0"/>
+  </joint>
+  <link name="tip_station_5mm_holder">
+    <visual>
+      <origin xyz="0 -0.0123 0" rpy="0 0 0"/>
+      <geometry>
+        <mesh filename="package://meca500_scene_description/meshes/onshape/_3D_printed.stl"/>
+      </geometry>
+      <material name="holder_colour">
+        <color rgba="0.95 0.75 0.20 1.0"/>
+      </material>
+    </visual>
+    <collision>
+      <origin xyz="0 -0.0123 0" rpy="0 0 0"/>
+      <geometry>
+        <mesh filename="package://meca500_scene_description/meshes/onshape/_3D_printed.stl"/>
+      </geometry>
+    </collision>
+  </link>
+  <joint name="tip_station_5mm_coupling_base_to_holder" type="fixed">
+    <parent link="tip_station_5mm_coupling_base"/>
+    <child link="tip_station_5mm_holder"/>
+    <origin xyz="-0.006 0 0.005"
+            rpy="-1.5708 0 1.5708"/>
+  </joint>
+  <!-- ========================================================= -->
+  <!-- Breadboard attachment                                     -->
+  <!-- ========================================================= -->
+  <joint name="bench_to_breadboard" type="fixed">
+    <parent link="bench_frame"/>
+    <child link="bench_breadboard"/>
+    <origin xyz="0 0 0"
+            rpy="-1.5708 0 0"/>
+  </joint>
 <xacro:meca500 parent="bench_breadboard">
   <!--
@@ -198,8 +303,8 @@
   <!--   part_1_2   -> tools_mount                              -->
   <!--   part_1   -> laser_sensor_mount                         -->
-  <!--   8777405    -> laser_sensor                             -->
+  <!--   _8777405    -> laser_sensor                            -->
   <!--   Force_sensor -> force_sensor                           -->
   <!--   part_1_3   -> april_tag_mount                          -->
-  <!--   part_1_10   -> force_poker                             -->
+  <!--   part_1_1   -> force_poker                              -->
   <!--                                                          -->
   <!-- NOTE: link_6 <-> CAD l6 frame equivalence must be        -->
@@ -218,4 +323,11 @@
       </material>
     </visual>
+    <collision>
+    <origin xyz="-0.00548008 0 -0.00548008"
+            rpy="0 0 0"/>
+    <geometry>
+      <mesh filename="package://meca500_scene_description/meshes/onshape/tools_mount.stl"/>
+    </geometry>
+    </collision>
   </link>
   <joint name="link_6_to_tools_mount" type="fixed">
@@ -237,4 +349,11 @@
       </material>
     </visual>
+    <collision>
+      <origin xyz="-0.00273616 -0.00751754 -0.0575"
+              rpy="0 0 0"/>
+      <geometry>
+        <mesh filename="package://meca500_scene_description/meshes/onshape/laser_sensor_mount.stl"/>
+      </geometry>
+    </collision>
   </link>
   <joint name="tools_mount_to_laser_sensor_mount" type="fixed">
@@ -256,4 +375,11 @@
       </material>
     </visual>
+    <collision>
+      <origin xyz="-0.01 -0.0028 0.0215"
+              rpy="0 0 0"/>
+      <geometry>
+        <mesh filename="package://meca500_scene_description/meshes/onshape/laser_sensor.stl"/>
+      </geometry>
+    </collision>
   </link>
   <joint name="laser_sensor_mount_to_laser_sensor" type="fixed">
@@ -275,4 +401,11 @@
       </material>
     </visual>
+    <collision>
+      <origin xyz="0.0277 0 0"
+              rpy="0 0 0"/>
+      <geometry>
+        <mesh filename="package://meca500_scene_description/meshes/onshape/force_sensor.stl"/>
+      </geometry>
+    </collision>
   </link>
   <joint name="tools_mount_to_force_sensor" type="fixed">
@@ -294,4 +427,11 @@
       </material>
     </visual>
+    <collision>
+      <origin xyz="-0.004 0 -0.03375"
+              rpy="0 0 0"/>
+      <geometry>
+        <mesh filename="package://meca500_scene_description/meshes/onshape/force_poker.stl"/>
+      </geometry>
+    </collision>
   </link>
   <joint name="force_sensor_to_force_poker" type="fixed">
@@ -313,4 +453,11 @@
       </material>
     </visual>
+    <collision>
+      <origin xyz="0 0.01 0"
+              rpy="0 0 0"/>
+      <geometry>
+        <mesh filename="package://meca500_scene_description/meshes/onshape/april_tag_mount.stl"/>
+      </geometry>
+    </collision>
   </link>
   <joint name="tools_mount_to_april_tag_mount" type="fixed">
