Commit message: Separate bench visuals from environment collision model

File: src/meca500_scene_description/urdf/scene.urdf.xacro (robot description, xacro)
@@ -2,295 +2,35 @@
 <robot name="helico_bench" xmlns:xacro="http://www.ros.org/wiki/xacro">
   <!-- Trusted Meca500 robot model -->
-  <xacro:include filename="$(find meca500_description)/urdf/meca500_macro.xacro"/>
-  <!-- Global reference frame for the Helico bench CAD -->
-  <link name="world"/>
-  <link name="bench_frame"/>
-  <joint name="world_to_bench" type="fixed">
-    <parent link="world"/>
-    <child link="bench_frame"/>
-    <origin xyz="0 0 0" rpy="0 0 0"/>
-  </joint>
-  <!--
-    Helico bench breadboard.
-    This mesh comes from the original Onshape URDF export and is the
-    authoritative geometric reference for positioning the physical bench.
-    No manually tuned RViz offset is applied here.
-  -->
-  <link name="bench_breadboard">
-    <visual>
-      <origin xyz="0 -0.0127 0" rpy="0 0 0"/>
-      <geometry>
-        <mesh filename="package://meca500_scene_description/meshes/onshape/MB3060_M___Aluminium_Breadboard_300_x_600_x_12_7mm_MB3030_M_1.stl"/>
-      </geometry>
-      <material name="breadboard_grey">
-        <color rgba="0.55 0.55 0.55 1.0"/>
-      </material>
-    </visual>
-    <collision>
-      <origin xyz="0 -0.0127 0" rpy="0 0 0"/>
-      <geometry>
-        <mesh filename="package://meca500_scene_description/meshes/onshape/MB3060_M___Aluminium_Breadboard_300_x_600_x_12_7mm_MB3030_M_1.stl"/>
-      </geometry>
-    </collision>
-  </link>
-  <!-- ========================================================= -->
-  <!-- Helico balloon tip stations                              -->
-  <!--                                                          -->
-  <!-- Ordered physically from robot-right to robot-left:        -->
-  <!--   3.5 mm -> 4 mm -> 5 mm                                 -->
-  <!--                                                          -->
-  <!-- Current station geometry is a PLACEHOLDER representation. -->
-  <!-- Repeated CAD meshes are used where the final Onshape CAD  -->
-  <!-- has not yet been completed.                               -->
-  <!--                                                          -->
-  <!-- Final station geometry should be updated from the latest  -->
-  <!-- Onshape assembly when available.                          -->
-  <!--                                                          -->
-  <!-- Helico CAD mapping:                                       -->
-  <!--   base_1 -> 3.5 mm station                                -->
-  <!--   base   -> 4 mm station                                  -->
-  <!--   base_2 -> 5 mm station                                  -->
-  <!-- ========================================================= -->
-  <!-- ========================================================= -->
-  <!-- 3.5 mm tip station                                        -->
-  <!-- Robot-right station                                       -->
-  <!-- ========================================================= -->
-  <link name="tip_station_3p5mm_base">
-    <visual>
-      <origin xyz="-0.0125 0.0125 0.025" rpy="0 0 0"/>
-      <geometry>
-        <mesh filename="package://meca500_scene_description/meshes/onshape/Base.stl"/>
-      </geometry>
-      <material name="base_colour">
-        <color rgba="0.4 0.7 0.9 1.0"/>
-      </material>
-    </visual>
-    <collision>
-      <origin xyz="-0.0125 0.0125 0.025" rpy="0 0 0"/>
-      <geometry>
-        <mesh filename="package://meca500_scene_description/meshes/onshape/Base.stl"/>
-      </geometry>
-    </collision>
-  </link>
-  <joint name="breadboard_to_tip_station_3p5mm_base" type="fixed">
-    <parent link="bench_breadboard"/>
-    <child link="tip_station_3p5mm_base"/>
-    <origin xyz="-0.0125 -0.0127 -0.0875"
-            rpy="1.5708 0 0"/>
-  </joint>
-  <link name="tip_station_3p5mm_coupling_base">
-    <visual>
-      <origin xyz="-0.006 0 0" rpy="0 0 0"/>
-      <geometry>
-        <mesh filename="package://meca500_scene_description/meshes/onshape/Coupling_base.stl"/>
-      </geometry>
-      <material name="coupling_colour">
-        <color rgba="0.1 0.3 0.8 1.0"/>
-      </material>
-    </visual>
-    <collision>
-      <origin xyz="-0.006 0 0" rpy="0 0 0"/>
-      <geometry>
-        <mesh filename="package://meca500_scene_description/meshes/onshape/Coupling_base.stl"/>
-      </geometry>
-    </collision>
-  </link>
-  <joint name="tip_station_3p5mm_base_to_coupling_base" type="fixed">
-    <parent link="tip_station_3p5mm_base"/>
-    <child link="tip_station_3p5mm_coupling_base"/>
-    <origin xyz="-0.0065 0.0125 0.025"
-            rpy="0 0 0"/>
-  </joint>
-  <link name="tip_station_3p5mm_holder">
-    <visual>
-      <origin xyz="0 -0.0123 0" rpy="0 0 0"/>
-      <geometry>
-        <mesh filename="package://meca500_scene_description/meshes/onshape/_3D_printed.stl"/>
-      </geometry>
-      <material name="holder_colour">
-        <color rgba="0.95 0.75 0.20 1.0"/>
-      </material>
-    </visual>
-    <collision>
-      <origin xyz="0 -0.0123 0" rpy="0 0 0"/>
-      <geometry>
-        <mesh filename="package://meca500_scene_description/meshes/onshape/_3D_printed.stl"/>
-      </geometry>
-    </collision>
-  </link>
-  <joint name="tip_station_3p5mm_coupling_base_to_holder" type="fixed">
-    <parent link="tip_station_3p5mm_coupling_base"/>
-    <child link="tip_station_3p5mm_holder"/>
-    <origin xyz="-0.006 0 0.005"
-            rpy="-1.5708 0 1.5708"/>
-  </joint>
-  <!-- ========================================================= -->
-  <!-- 4 mm tip station                                          -->
-  <!-- Middle station                                            -->
-  <!-- ========================================================= -->
-  <link name="tip_station_4mm_base">
-    <visual>
-      <origin xyz="0.0125 0.0125 0.025" rpy="0 0 0"/>
-      <geometry>
-        <mesh filename="package://meca500_scene_description/meshes/onshape/Base.stl"/>
-      </geometry>
-      <material name="base_colour">
-        <color rgba="0.4 0.7 0.9 1.0"/>
-      </material>
-    </visual>
-    <collision>
-      <origin xyz="0.0125 0.0125 0.025" rpy="0 0 0"/>
-      <geometry>
-        <mesh filename="package://meca500_scene_description/meshes/onshape/Base.stl"/>
-      </geometry>
-    </collision>
-  </link>
-  <joint name="breadboard_to_tip_station_4mm_base" type="fixed">
-    <parent link="bench_breadboard"/>
-    <child link="tip_station_4mm_base"/>
-    <origin xyz="-0.0375 -0.0127 -0.0125"
-            rpy="1.5708 0 0"/>
-  </joint>
-  <link name="tip_station_4mm_coupling_base">
-    <visual>
-      <origin xyz="-0.006 0 0" rpy="0 0 0"/>
-      <geometry>
-        <mesh filename="package://meca500_scene_description/meshes/onshape/Coupling_base.stl"/>
-      </geometry>
-      <material name="coupling_colour">
-        <color rgba="0.1 0.3 0.8 1.0"/>
-      </material>
-    </visual>
-    <collision>
-      <origin xyz="-0.006 0 0" rpy="0 0 0"/>
-      <geometry>
-        <mesh filename="package://meca500_scene_description/meshes/onshape/Coupling_base.stl"/>
-      </geometry>
-    </collision>
-  </link>
-  <joint name="tip_station_4mm_base_to_coupling_base" type="fixed">
-    <parent link="tip_station_4mm_base"/>
-    <child link="tip_station_4mm_coupling_base"/>
-    <origin xyz="0.0185 0.0125 0.025"
-            rpy="0 0 0"/>
-  </joint>
-  <link name="tip_station_4mm_holder">
-    <visual>
-      <origin xyz="0 -0.0123 0" rpy="0 0 0"/>
-      <geometry>
-        <mesh filename="package://meca500_scene_description/meshes/onshape/_3D_printed.stl"/>
-      </geometry>
-      <material name="holder_colour">
-        <color rgba="0.95 0.75 0.20 1.0"/>
-      </material>
-    </visual>
-    <collision>
-      <origin xyz="0 -0.0123 0" rpy="0 0 0"/>
-      <geometry>
-        <mesh filename="package://meca500_scene_description/meshes/onshape/_3D_printed.stl"/>
-      </geometry>
-    </collision>
-  </link>
-  <joint name="tip_station_4mm_coupling_base_to_holder" type="fixed">
-    <parent link="tip_station_4mm_coupling_base"/>
-    <child link="tip_station_4mm_holder"/>
-    <origin xyz="-0.006 0 0.005"
-            rpy="-1.5708 0 1.5708"/>
-  </joint>
-  <!-- ========================================================= -->
-  <!-- 5 mm tip station                                          -->
-  <!-- Robot-left station                                        -->
-  <!--                                                          -->
-  <!-- PLACEHOLDER: coupling and holder reuse the existing        -->
-  <!-- station meshes until final Onshape CAD is available.       -->
-  <!-- ========================================================= -->
-  <link name="tip_station_5mm_base">
-    <visual>
-      <origin xyz="-0.0125 0.0125 0.025" rpy="0 0 0"/>
-      <geometry>
-        <mesh filename="package://meca500_scene_description/meshes/onshape/Base.stl"/>
-      </geometry>
-      <material name="base_colour">
-        <color rgba="0.4 0.7 0.9 1.0"/>
-      </material>
-    </visual>
-    <collision>
-      <origin xyz="-0.0125 0.0125 0.025" rpy="0 0 0"/>
-      <geometry>
-        <mesh filename="package://meca500_scene_description/meshes/onshape/Base.stl"/>
-      </geometry>
-    </collision>
-  </link>
-  <joint name="breadboard_to_tip_station_5mm_base" type="fixed">
-    <parent link="bench_breadboard"/>
-    <child link="tip_station_5mm_base"/>
-    <origin xyz="-0.0125 -0.0127 0.0625"
-            rpy="1.5708 0 0"/>
-  </joint>
-  <link name="tip_station_5mm_coupling_base">
-    <visual>
-      <origin xyz="-0.006 0 0" rpy="0 0 0"/>
-      <geometry>
-        <mesh filename="package://meca500_scene_description/meshes/onshape/Coupling_base.stl"/>
-      </geometry>
-      <material name="coupling_colour">
-        <color rgba="0.1 0.3 0.8 1.0"/>
-      </material>
-    </visual>
-    <collision>
-      <origin xyz="-0.006 0 0" rpy="0 0 0"/>
-      <geometry>
-        <mesh filename="package://meca500_scene_description/meshes/onshape/Coupling_base.stl"/>
-      </geometry>
-    </collision>
-  </link>
-  <joint name="tip_station_5mm_base_to_coupling_base" type="fixed">
-    <parent link="tip_station_5mm_base"/>
-    <child link="tip_station_5mm_coupling_base"/>
-    <origin xyz="-0.0065 0.0125 0.025"
-            rpy="0 0 0"/>
-  </joint>
-  <link name="tip_station_5mm_holder">
-    <visual>
-      <origin xyz="0 -0.0123 0" rpy="0 0 0"/>
-      <geometry>
-        <mesh filename="package://meca500_scene_description/meshes/onshape/_3D_printed.stl"/>
-      </geometry>
-      <material name="holder_colour">
-        <color rgba="0.95 0.75 0.20 1.0"/>
-      </material>
-    </visual>
-    <collision>
-      <origin xyz="0 -0.0123 0" rpy="0 0 0"/>
-      <geometry>
-        <mesh filename="package://meca500_scene_description/meshes/onshape/_3D_printed.stl"/>
-      </geometry>
-    </collision>
-  </link>
-  <joint name="tip_station_5mm_coupling_base_to_holder" type="fixed">
-    <parent link="tip_station_5mm_coupling_base"/>
-    <child link="tip_station_5mm_holder"/>
-    <origin xyz="-0.006 0 0.005"
-            rpy="-1.5708 0 1.5708"/>
-  </joint>
-  <!-- ========================================================= -->
-  <!-- Breadboard attachment                                     -->
-  <!-- ========================================================= -->
-  <joint name="bench_to_breadboard" type="fixed">
-    <parent link="bench_frame"/>
-    <child link="bench_breadboard"/>
-    <origin xyz="0 0 0"
-            rpy="-1.5708 0 0"/>
-  </joint>
-<xacro:meca500 parent="bench_breadboard">
-  <!--
-    Trusted ROS Meca500 kinematic model positioned using Helico's CAD.
-    Placement derived from rigid registration of Helico's Base_1.stl
-    against the trusted ROS Meca500 base mesh.
-    Do not tune this transform manually in RViz.
-  -->
-  <origin xyz="-0.175 -0.0127 -0.025"
-          rpy="1.5708 0 0"/>
-</xacro:meca500>
+  <xacro:include filename="$(find meca500_description)/urdf/meca500_macro.xacro" />
+  <!-- Helico bench frames and visual environment -->
+  <xacro:include filename="$(find meca500_scene_description)/urdf/frames/bench_frames.xacro" />
+  <xacro:include filename="$(find meca500_scene_description)/urdf/visuals/breadboard_visual.xacro" />
+  <xacro:include filename="$(find meca500_scene_description)/urdf/visuals/station_visuals.xacro" />
+  <!-- Global root -->
+  <link name="world" />
+  <!-- Visual only. Collision version is loaded into MoveIt PlanningScene. -->
+  <xacro:breadboard_visual parent="bench_breadboard" />
+  <!-- 3.5 mm station -->
+  <xacro:station_visual
+    prefix="tip_station_3p5mm"
+    parent="tip_station_3p5mm_frame"
+    base_visual_x="-0.0125"
+    coupling_x="-0.0065" />
+  <!-- 4 mm station -->
+  <xacro:station_visual
+    prefix="tip_station_4mm"
+    parent="tip_station_4mm_frame"
+    base_visual_x="0.0125"
+    coupling_x="0.0185" />
+  <!-- 5 mm station -->
+  <xacro:station_visual
+    prefix="tip_station_5mm"
+    parent="tip_station_5mm_frame"
+    base_visual_x="-0.0125"
+    coupling_x="-0.0065" />
+  <xacro:meca500 parent="bench_breadboard">
+    <origin xyz="-0.175 -0.0127 -0.025"
+      rpy="1.5708 0 0" />
+  </xacro:meca500>
   <!-- ========================================================= -->
   <!-- Link 6 measurement tool                                  -->
@@ -315,25 +55,25 @@
     <visual>
       <origin xyz="-0.00548008 0 -0.00548008"
-              rpy="0 0 0"/>
-      <geometry>
-        <mesh filename="package://meca500_scene_description/meshes/onshape/tools_mount.stl"/>
+        rpy="0 0 0" />
+      <geometry>
+        <mesh filename="package://meca500_scene_description/meshes/onshape/tools_mount.stl" />
       </geometry>
       <material name="tools_mount_colour">
-        <color rgba="0.682353 0.333333 0.737255 1"/>
-      </material>
-    </visual>
-    <collision>
-    <origin xyz="-0.00548008 0 -0.00548008"
-            rpy="0 0 0"/>
-    <geometry>
-      <mesh filename="package://meca500_scene_description/meshes/onshape/tools_mount.stl"/>
-    </geometry>
+        <color rgba="0.682353 0.333333 0.737255 1" />
+      </material>
+    </visual>
+    <collision>
+      <origin xyz="-0.00548008 0 -0.00548008"
+        rpy="0 0 0" />
+      <geometry>
+        <mesh filename="package://meca500_scene_description/meshes/onshape/tools_mount.stl" />
+      </geometry>
     </collision>
   </link>
   <joint name="link_6_to_tools_mount" type="fixed">
-    <parent link="link_6"/>
-    <child link="tools_mount"/>
+    <parent link="link_6" />
+    <child link="tools_mount" />
     <origin xyz="-0.00548008 0.00548008 0"
-            rpy="-1.5708 0 1.5708"/>
+      rpy="-1.5708 0 1.5708" />
   </joint>
   <!-- Laser mounting/support component -->
@@ -341,25 +81,25 @@
     <visual>
       <origin xyz="-0.00273616 -0.00751754 -0.0575"
-              rpy="0 0 0"/>
-      <geometry>
-        <mesh filename="package://meca500_scene_description/meshes/onshape/laser_sensor_mount.stl"/>
+        rpy="0 0 0" />
+      <geometry>
+        <mesh filename="package://meca500_scene_description/meshes/onshape/laser_sensor_mount.stl" />
       </geometry>
       <material name="laser_sensor_mount_colour">
-        <color rgba="0.729412 0.25098 0.105882 1"/>
+        <color rgba="0.729412 0.25098 0.105882 1" />
       </material>
     </visual>
     <collision>
       <origin xyz="-0.00273616 -0.00751754 -0.0575"
-              rpy="0 0 0"/>
-      <geometry>
-        <mesh filename="package://meca500_scene_description/meshes/onshape/laser_sensor_mount.stl"/>
+        rpy="0 0 0" />
+      <geometry>
+        <mesh filename="package://meca500_scene_description/meshes/onshape/laser_sensor_mount.stl" />
       </geometry>
     </collision>
   </link>
   <joint name="tools_mount_to_laser_sensor_mount" type="fixed">
-    <parent link="tools_mount"/>
-    <child link="laser_sensor_mount"/>
+    <parent link="tools_mount" />
+    <child link="laser_sensor_mount" />
     <origin xyz="0.00203746 -0.005 0.0247125"
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
Commit message: Align Link 6 tooling and add joint pose support

File: src/meca500_scene_description/urdf/scene.urdf.xacro (robot description, xacro)
@@ -74,6 +74,6 @@
     <parent link="link_6" />
     <child link="tools_mount" />
-    <origin xyz="-0.00548008 0.00548008 0"
-      rpy="-1.5708 0 1.5708" />
+    <origin xyz="0.00548008 0.00548008 0"
+      rpy="-1.5708 0 0" />
   </joint>
   <!-- Laser mounting/support component -->
